File: control-logic.sch (KiCad schematic (older format))
At the start: 34 parts, among them U1 STM32F072R, U2 MCP2562, X1 8.000 MHz

Commit message: KiCad 4 migration changes, mostly
Parts:
- C1, C2, C3, C4, C5, C6, C7, C8, C9: symbol C -> C-RESCUE-servo-module-pcb-v1
- HB1, PG1: symbol LED -> LED-RESCUE-servo-module-pcb-v1
- R1, R10, R11, R12, R13, R14, R2, R3, R4, R5, R6, R7, R8, R9: symbol R -> R-RESCUE-servo-module-pcb-v1
Changed lines of the file:
@@
 EESchema Schematic File Version 2
+LIBS:servo-module-pcb-v1-rescue
 LIBS:power
 LIBS:device
@@
 LIBS:memory
 LIBS:xilinx
-LIBS:special
 LIBS:microcontrollers
 LIBS:dsp
@@
 $EndComp
 $Comp
-L R R14
+L R-RESCUE-servo-module-pcb-v1 R14
 U 1 1 5325B4BA
 P 9650 6200
@@
 $EndComp
 $Comp
-L R R13
+L R-RESCUE-servo-module-pcb-v1 R13
 U 1 1 5325B4C9
 P 9450 6200
@@
 $EndComp
 $Comp
-L R R12
+L R-RESCUE-servo-module-pcb-v1 R12
 U 1 1 5325B4D8
 P 9250 6200
@@
 $EndComp
 $Comp
-L R R11
+L R-RESCUE-servo-module-pcb-v1 R11
 U 1 1 5325B4E7
 P 9050 6200
@@
 $EndComp
 $Comp
-L R R10
+L R-RESCUE-servo-module-pcb-v1 R10
 U 1 1 5325B4F6
 P 8850 6200
@@
 $EndComp
 $Comp
-L R R9
+L R-RESCUE-servo-module-pcb-v1 R9
 U 1 1 5325B505
 P 8650 6200
@@
 $EndComp
 $Comp
-L R R8
+L R-RESCUE-servo-module-pcb-v1 R8
 U 1 1 5325B514
 P 8450 6200
@@
 $EndComp
 $Comp
-L R R7
+L R-RESCUE-servo-module-pcb-v1 R7
 U 1 1 5325B523
 P 8250 6200
@@
 $EndComp
 $Comp
-L GND #PWR10
+L GND-RESCUE-servo-module-pcb-v1 #PWR10
 U 1 1 5325BA22
 P 9050 6650
@@
 $EndComp
 $Comp
-L GND #PWR8
+L GND-RESCUE-servo-module-pcb-v1 #PWR8
 U 1 1 53262BD9
 P 3050 5600
@@
 $EndComp
 $Comp
-L C C2
+L C-RESCUE-servo-module-pcb-v1 C2
 U 1 1 53264A23
 P 1500 2000
@@
 $EndComp
 $Comp
-L C C1
+L C-RESCUE-servo-module-pcb-v1 C1
 U 1 1 53264A32
 P 1500 1400
@@
 $EndComp
 $Comp
-L GND #PWR2
+L GND-RESCUE-servo-module-pcb-v1 #PWR2
 U 1 1 53264B7B
 P 1200 2100
@@
 $EndComp
 $Comp
-L LED PG1
+L LED-RESCUE-servo-module-pcb-v1 PG1
 U 1 1 53267B24
 P 10100 1250
@@
 $EndComp
 $Comp
-L LED HB1
+L LED-RESCUE-servo-module-pcb-v1 HB1
 U 1 1 53267B33
 P 9800 1250
@@
 $EndComp
 $Comp
-L R R2
+L R-RESCUE-servo-module-pcb-v1 R2
 U 1 1 53267B42
 P 8500 1100
@@
 $EndComp
 $Comp
-L R R1
+L R-RESCUE-servo-module-pcb-v1 R1
 U 1 1 53267B51
 P 8050 1100
@@
 $EndComp
 $Comp
-L R R4
+L R-RESCUE-servo-module-pcb-v1 R4
 U 1 1 53267B60
 P 10100 1800
@@
 $EndComp
 $Comp
-L R R3
+L R-RESCUE-servo-module-pcb-v1 R3
 U 1 1 53267B6F
 P 9800 1800
@@
 $EndComp
 $Comp
-L C C3
+L C-RESCUE-servo-module-pcb-v1 C3
 U 1 1 53267B9C
 P 6350 6150
@@
 $EndComp
 $Comp
-L C C4
+L C-RESCUE-servo-module-pcb-v1 C4
 U 1 1 53267BAB
 P 6600 6150
@@
 $EndComp
 $Comp
-L C C5
+L C-RESCUE-servo-module-pcb-v1 C5
 U 1 1 53267BBA
 P 6850 6150
@@
 $EndComp
 $Comp
-L C C6
+L C-RESCUE-servo-module-pcb-v1 C6
 U 1 1 53267BC9
 P 7100 6150
@@
 $EndComp
 $Comp
-L C C7
+L C-RESCUE-servo-module-pcb-v1 C7
 U 1 1 53267BD8
 P 7350 6150
@@
 $EndComp
 $Comp
-L GND #PWR9
+L GND-RESCUE-servo-module-pcb-v1 #PWR9
 U 1 1 53268402
 P 6350 6550
@@
 LOCAL_3V3
 $Comp
-L GND #PWR3
+L GND-RESCUE-servo-module-pcb-v1 #PWR3
 U 1 1 53268FE5
 P 8050 2250
@@
 $EndComp
 $Comp
-L GND #PWR4
+L GND-RESCUE-servo-module-pcb-v1 #PWR4
 U 1 1 532697A4
 P 9950 2250
@@
 POWER_GOOD
 $Comp
-L GND #PWR5
+L GND-RESCUE-servo-module-pcb-v1 #PWR5
 U 1 1 5326A151
 P 7850 3100
@@
 TXD
 $Comp
-L GND #PWR6
+L GND-RESCUE-servo-module-pcb-v1 #PWR6
 U 1 1 5326B790
 P 10000 3100
@@
 SDA
 $Comp
-L GND #PWR7
+L GND-RESCUE-servo-module-pcb-v1 #PWR7
 U 1 1 533CA56F
 P 9100 4150
@@
 $EndComp
 $Comp
-L R R6
+L R-RESCUE-servo-module-pcb-v1 R6
 U 1 1 533CAC4E
 P 8950 3650
@@
 $EndComp
 $Comp
-L R R5
+L R-RESCUE-servo-module-pcb-v1 R5
 U 1 1 533CAE0E
 P 8750 3650
@@
 $EndComp
 $Comp
-L GND #PWR11
+L GND-RESCUE-servo-module-pcb-v1 #PWR11
 U 1 1 54EC01AF
 P 2200 7650
@@
 LOCAL_5V
 $Comp
-L C C8
+L C-RESCUE-servo-module-pcb-v1 C8
 U 1 1 54EC1BB5
 P 3750 7250
@@
 $EndComp
 $Comp
-L C C9
+L C-RESCUE-servo-module-pcb-v1 C9
 U 1 1 54EC1E37
 P 4050 7250
@@
 $EndComp
 $Comp
-L GND #PWR12
+L GND-RESCUE-servo-module-pcb-v1 #PWR12
 U 1 1 54EC1E75
 P 3900 7650
