File: power-supply.sch (KiCad schematic (older format))
At the start: 30 parts, among them U5 AP3513E, U6 ZXCT1107SA-7, U7 AP1117IE33G

Commit message: KiCad 4 migration changes, mostly
Parts:
- C12, C13, C18, C19, C22: symbol C -> C-RESCUE-servo-module-pcb-v1
- C14, C15, C16, C17, C20, C21: symbol CP -> CP-RESCUE-servo-module-pcb-v1
- D1, D2, D3: symbol LED -> LED-RESCUE-servo-module-pcb-v1
- R31, R32, R33, R34, R35, R36, R37, R38, R39, R40, R41: symbol R -> R-RESCUE-servo-module-pcb-v1
Changed lines of the file:
@@
 EESchema Schematic File Version 2
+LIBS:servo-module-pcb-v1-rescue
 LIBS:power
 LIBS:device
@@
 LIBS:memory
 LIBS:xilinx
-LIBS:special
 LIBS:microcontrollers
 LIBS:dsp
@@
 $EndComp
 $Comp
-L GND #PWR28
+L GND-RESCUE-servo-module-pcb-v1 #PWR28
 U 1 1 5323D81B
 P 7800 4450
@@
 $EndComp
 Wire Wire Line
-	7800 4050 7800 4350
-Wire Wire Line
-	7800 4350 7800 4450
-Wire Wire Line
-	8200 3750 8350 3750
-Wire Wire Line
-	8350 3750 8500 3750
-$Comp
-L +3.3V #PWR27
+	7800 4050 7800 4450
+Wire Wire Line
+	8200 3750 8500 3750
+$Comp
+L +3.3V-RESCUE-servo-module-pcb-v1 #PWR27
 U 1 1 5323D834
 P 8350 3650
+AR Path="/5323D834" Ref="#PWR27"  Part="1"
+AR Path="/5311518E/5323D834" Ref="#PWR27"  Part="1"
 F 0 "#PWR27" H 8350 3610 30  0001 C CNN
 F 1 "+3.3V" H 8350 3760 30  0000 C CNN
@@
 $EndComp
 Wire Wire Line
-	8350 3650 8350 3750
-Wire Wire Line
-	8350 3750 8350 3850
+	8350 3650 8350 3850
 Connection ~ 8350 3750
 Wire Wire Line
-	1900 950  2100 950
-Wire Wire Line
-	2100 950  2200 950
-Wire Wire Line
-	2200 950  2500 950
-Wire Wire Line
-	2500 950  5300 950
+	1900 950  5300 950
 Connection ~ 2100 950
 $Comp
-L CP C21
+L CP-RESCUE-servo-module-pcb-v1 C21
 U 1 1 5323D89B
 P 7300 4050
@@
 	8350 4350 8350 4250
 Wire Wire Line
-	7300 4350 7800 4350
-Wire Wire Line
-	7800 4350 8350 4350
+	7300 4350 8350 4350
 Connection ~ 7800 4350
 Wire Wire Line
 	7300 4350 7300 4250
 Wire Wire Line
-	7300 3650 7300 3750
-Wire Wire Line
-	7300 3750 7300 3850
+	7300 3650 7300 3850
 Connection ~ 7300 3750
 $Comp
-L C C22
+L C-RESCUE-servo-module-pcb-v1 C22
 U 1 1 5323DB4D
 P 8350 4050
@@
 $EndComp
 $Comp
-L R R39
+L R-RESCUE-servo-module-pcb-v1 R39
 U 1 1 5323DD18
 P 9400 5350
@@
 $EndComp
 $Comp
-L R R40
+L R-RESCUE-servo-module-pcb-v1 R40
 U 1 1 5323DD27
 P 9700 5350
@@
 $EndComp
 $Comp
-L R R41
+L R-RESCUE-servo-module-pcb-v1 R41
 U 1 1 5323DD36
 P 10000 5350
@@
 $EndComp
 $Comp
-L LED D1
+L LED-RESCUE-servo-module-pcb-v1 D1
 U 1 1 5323DD59
 P 9400 5900
@@
 $EndComp
 $Comp
-L LED D2
+L LED-RESCUE-servo-module-pcb-v1 D2
 U 1 1 5323DD77
 P 9700 5900
@@
 $EndComp
 $Comp
-L LED D3
+L LED-RESCUE-servo-module-pcb-v1 D3
 U 1 1 5323DD86
 P 10000 5900
@@
 	9400 6100 9400 6200
 $Comp
-L GND #PWR32
+L GND-RESCUE-servo-module-pcb-v1 #PWR32
 U 1 1 5323DED8
 P 9550 6300
@@
 Connection ~ 9550 6200
 $Comp
-L +3.3V #PWR31
+L +3.3V-RESCUE-servo-module-pcb-v1 #PWR31
 U 1 1 5323DF0D
 P 10000 5000
+AR Path="/5323DF0D" Ref="#PWR31"  Part="1"
+AR Path="/5311518E/5323DF0D" Ref="#PWR31"  Part="1"
 F 0 "#PWR31" H 10000 4960 30  0001 C CNN
 F 1 "+3.3V" H 10000 5110 30  0000 C CNN
@@
 ISERVO_SENSE_OUT
 $Comp
-L R R32
+L R-RESCUE-servo-module-pcb-v1 R32
 U 1 1 5325ED8A
 P 7800 1050
@@
 $EndComp
 Wire Wire Line
-	8050 1050 8100 1050
-Wire Wire Line
-	8100 1050 8450 1050
+	8050 1050 8450 1050
 Wire Wire Line
 	8100 1200 8100 1050
@@
 $EndComp
 $Comp
-L R R36
+L R-RESCUE-servo-module-pcb-v1 R36
 U 1 1 5325F162
 P 7800 2550
@@
 $EndComp
 Wire Wire Line
-	7800 2200 7800 2250
-Wire Wire Line
-	7800 2250 7800 2300
-$Comp
-L GND #PWR24
+	7800 2200 7800 2300
+$Comp
+L GND-RESCUE-servo-module-pcb-v1 #PWR24
 U 1 1 5325F1C0
 P 7800 2900
@@
 Connection ~ 7800 2250
 $Comp
-L R R37
+L R-RESCUE-servo-module-pcb-v1 R37
 U 1 1 5325F7A5
 P 2550 2600
@@
 	2100 2600 2300 2600
 Wire Wire Line
-	2800 2600 2950 2600
-Wire Wire Line
-	2950 2600 3300 2600
-Wire Wire Line
-	3300 2600 3600 2600
-$Comp
-L R R38
+	2800 2600 3600 2600
+$Comp
+L R-RESCUE-servo-module-pcb-v1 R38
 U 1 1 5325F83D
 P 2950 3000
@@
 $EndComp
 $Comp
-L GND #PWR25
+L GND-RESCUE-servo-module-pcb-v1 #PWR25
 U 1 1 5325F856
 P 2950 3450
@@
 $EndComp
 Wire Wire Line
-	2950 3250 2950 3350
-Wire Wire Line
-	2950 3350 2950 3450
+	2950 3250 2950 3450
 Wire Wire Line
 	2950 2750 2950 2600
 Connection ~ 2950 2600
 $Comp
-L CP C20
+L CP-RESCUE-servo-module-pcb-v1 C20
 U 1 1 5325F8F3
 P 3300 3000
@@
 LRC-LR1206LF-01-R075F
 Wire Wire Line
-	9400 6200 9550 6200
-Wire Wire Line
-	9550 6200 9700 6200
-Wire Wire Line
-	9700 6200 10000 6200
+	9400 6200 10000 6200
 $Comp
 L AP3513E U5
@@
 $EndComp
 $Comp
-L GND #PWR21
+L GND-RESCUE-servo-module-pcb-v1 #PWR21
 U 1 1 5575F4E6
 P 5300 1750
@@
 	5200 1550 5300 1550
 Wire Wire Line
-	5300 1550 5300 1650
-Wire Wire Line
-	5300 1650 5300 1750
+	5300 1550 5300 1750
 Wire Wire Line
 	5200 1650 5300 1650
 Connection ~ 5300 1650
 $Comp
-L R R31
+L R-RESCUE-servo-module-pcb-v1 R31
 U 1 1 5575F4F0
 P 4600 1050
@@
 $EndComp
 $Comp
-L C C19
+L C-RESCUE-servo-module-pcb-v1 C19
 U 1 1 5575F4F7
 P 3600 1650
@@
 $EndComp
 $Comp
-L R R33
+L R-RESCUE-servo-module-pcb-v1 R33
 U 1 1 5575F4FE
 P 3050 1650
@@
 $EndComp
 $Comp
-L C C18
+L C-RESCUE-servo-module-pcb-v1 C18
 U 1 1 5575F505
 P 3350 1500
@@
 $EndComp
 $Comp
-L C C12
+L C-RESCUE-servo-module-pcb-v1 C12
 U 1 1 5575F50C
 P 3350 1250
@@
 	4000 1550 3850 1550
 Wire Wire Line
-	3850 1500 3850 1550
-Wire Wire Line
-	3850 1550 3850 1650
+	3850 1500 3850 1650
 Wire Wire Line
 	3850 1650 3800 1650
@@
 	3400 1650 3300 1650
 $Comp
-L GND #PWR23
+L GND-RESCUE-servo-module-pcb-v1 #PWR23
 U 1 1 5575F51C
 P 2700 1950
@@
 $EndComp
 Wire Wire Line
-	2700 1250 2700 1500
-Wire Wire Line
-	2700 1500 2700 1650
-Wire Wire Line
-	2700 1650 2700 1850
-Wire Wire Line
-	2700 1850 2700 1950
+	2700 1250 2700 1950
 Wire Wire Line
 	2700 1250 3150 1250
@@
 Connection ~ 2700 1650
 $Comp
-L C C13
+L C-RESCUE-servo-module-pcb-v1 C13
 U 1 1 5575F528
 P 5600 1250
@@
 	5200 1250 5400 1250
 Wire Wire Line
-	5200 1450 5900 1450
-Wire Wire Line
-	5900 1450 6000 1450
+	5200 1450 6000 1450
 Wire Wire Line
 	5900 1450 5900 1250
@@
 	4850 1050 5300 1050
 Wire Wire Line
-	5300 950  5300 1050
-Wire Wire Line
-	5300 1050 5300 1350
+	5300 950  5300 1350
 Wire Wire Line
 	5300 1350 5200 1350
@@
 Connection ~ 5900 1450
 $Comp
-L R R34
+L R-RESCUE-servo-module-pcb-v1 R34
 U 1 1 5575F53F
 P 3050 1850
@@
 $EndComp
 $Comp
-L R R35
+L R-RESCUE-servo-module-pcb-v1 R35
 U 1 1 5575F546
 P 3750 1850
@@
 	3400 1750 3400 1850
 Wire Wire Line
-	3300 1850 3400 1850
-Wire Wire Line
-	3400 1850 3500 1850
+	3300 1850 3500 1850
 Connection ~ 3400 1850
 Wire Wire Line
-	2200 1850 2500 1850
-Wire Wire Line
-	2500 1850 2700 1850
-Wire Wire Line
-	2700 1850 2800 1850
+	2200 1850 2800 1850
 Connection ~ 2700 1850
 Wire Wire Line
 	6700 1850 4000 1850
 Wire Wire Line
-	6700 950  6700 1050
-Wire Wire Line
-	6700 1050 6700 1450
-Wire Wire Line
-	6700 1450 6700 1850
+	6700 950  6700 1850
 Wire Wire Line
 	6700 1450 6600 1450
@@
 $EndComp
 Wire Wire Line
-	2200 850  2200 950
-Wire Wire Line
-	2200 950  2200 1250
+	2200 850  2200 1250
 Connection ~ 5300 1050
 $Comp
-L CP C16
+L CP-RESCUE-servo-module-pcb-v1 C16
 U 1 1 5575F568
 P 2200 1450
@@
 $EndComp
 $Comp
-L CP C17
+L CP-RESCUE-servo-module-pcb-v1 C17
 U 1 1 5575F56F
 P 2500 1450
@@
 Connection ~ 2500 950
 $Comp
-L CP C14
+L CP-RESCUE-servo-module-pcb-v1 C14
 U 1 1 5575F57C
 P 6850 1350
@@
 $EndComp
 $Comp
-L CP C15
+L CP-RESCUE-servo-module-pcb-v1 C15
 U 1 1 5575F583
 P 7100 1350
@@
 $EndComp
 Wire Wire Line
-	6850 1550 6850 1650
-Wire Wire Line
-	6850 1650 6850 1750
+	6850 1550 6850 1750
 Wire Wire Line
 	6850 1650 7100 1650
@@
 	7100 1650 7100 1550
 Wire Wire Line
-	6700 1050 6850 1050
-Wire Wire Line
-	6850 1050 7100 1050
-Wire Wire Line
-	7100 1050 7250 1050
-Wire Wire Line
-	7250 1050 7500 1050
-Wire Wire Line
-	7500 1050 7550 1050
+	6700 1050 7550 1050
 Wire Wire Line
 	7100 1050 7100 1150
@@
 Connection ~ 6850 1050
 $Comp
-L GND #PWR22
+L GND-RESCUE-servo-module-pcb-v1 #PWR22
 U 1 1 5575F592
 P 6850 1750
