File: servo-driver.sch (KiCad schematic (older format))
At the start: 26 parts, among them P3 CONN_01X08, P4 CONN_01X08, P5 CONN_01X08, P6 CONN_01X08, P7 CONN_01X08, P8 CONN_01X08, U3 74HC245, U4 74HC245

Commit message: KiCad 4 migration changes, mostly
Parts:
- C10, C11: symbol C -> C-RESCUE-servo-module-pcb-v1
- R15, R16, R17, R18, R19, R20, R21, R22, R23, R24, R25, R26, R27, R28, R29, R30: symbol R -> R-RESCUE-servo-module-pcb-v1
Changed lines of the file:
@@
 EESchema Schematic File Version 2
+LIBS:servo-module-pcb-v1-rescue
 LIBS:power
 LIBS:device
@@
 LIBS:memory
 LIBS:xilinx
-LIBS:special
 LIBS:microcontrollers
 LIBS:dsp
@@
 	4450 3250 4250 3250
 $Comp
-L GND #PWR15
+L GND-RESCUE-servo-module-pcb-v1 #PWR15
 U 1 1 55758CD7
 P 5150 4500
@@
 	3250 2850 7350 2850
 $Comp
-L R R15
+L R-RESCUE-servo-module-pcb-v1 R15
 U 1 1 55758D17
 P 6200 3250
@@
 $EndComp
 $Comp
-L R R16
+L R-RESCUE-servo-module-pcb-v1 R16
 U 1 1 55758D77
 P 6600 3350
@@
 $EndComp
 $Comp
-L R R17
+L R-RESCUE-servo-module-pcb-v1 R17
 U 1 1 55758DA2
 P 6200 3450
@@
 $EndComp
 $Comp
-L R R18
+L R-RESCUE-servo-module-pcb-v1 R18
 U 1 1 55758DCE
 P 6600 3550
@@
 $EndComp
 $Comp
-L R R19
+L R-RESCUE-servo-module-pcb-v1 R19
 U 1 1 55758E0E
 P 6200 3650
@@
 $EndComp
 $Comp
-L R R20
+L R-RESCUE-servo-module-pcb-v1 R20
 U 1 1 55758E36
 P 6600 3750
@@
 $EndComp
 $Comp
-L R R21
+L R-RESCUE-servo-module-pcb-v1 R21
 U 1 1 55758E5D
 P 6200 3850
@@
 $EndComp
 $Comp
-L R R22
+L R-RESCUE-servo-module-pcb-v1 R22
 U 1 1 55758EA1
 P 6600 3950
@@
 Connection ~ 7850 3350
 $Comp
-L GND #PWR14
+L GND-RESCUE-servo-module-pcb-v1 #PWR14
 U 1 1 557595E9
 P 7850 4150
@@
 	4450 5350 4250 5350
 $Comp
-L GND #PWR18
+L GND-RESCUE-servo-module-pcb-v1 #PWR18
 U 1 1 55759ADF
 P 5150 6600
@@
 	5150 5300 5150 4950
 $Comp
-L R R23
+L R-RESCUE-servo-module-pcb-v1 R23
 U 1 1 55759AE8
 P 6200 5350
@@
 $EndComp
 $Comp
-L R R24
+L R-RESCUE-servo-module-pcb-v1 R24
 U 1 1 55759AEE
 P 6600 5450
@@
 $EndComp
 $Comp
-L R R25
+L R-RESCUE-servo-module-pcb-v1 R25
 U 1 1 55759AF4
 P 6200 5550
@@
 $EndComp
 $Comp
-L R R26
+L R-RESCUE-servo-module-pcb-v1 R26
 U 1 1 55759AFA
 P 6600 5650
@@
 $EndComp
 $Comp
-L R R27
+L R-RESCUE-servo-module-pcb-v1 R27
 U 1 1 55759B00
 P 6200 5750
@@
 $EndComp
 $Comp
-L R R28
+L R-RESCUE-servo-module-pcb-v1 R28
 U 1 1 55759B06
 P 6600 5850
@@
 $EndComp
 $Comp
-L R R29
+L R-RESCUE-servo-module-pcb-v1 R29
 U 1 1 55759B0C
 P 6200 5950
@@
 $EndComp
 $Comp
-L R R30
+L R-RESCUE-servo-module-pcb-v1 R30
 U 1 1 55759B12
 P 6600 6050
@@
 Connection ~ 7850 5450
 $Comp
-L GND #PWR17
+L GND-RESCUE-servo-module-pcb-v1 #PWR17
 U 1 1 55759B59
 P 7850 6250
@@
 Connection ~ 3700 4150
 $Comp
-L C C10
+L C-RESCUE-servo-module-pcb-v1 C10
 U 1 1 55767058
 P 3500 3600
@@
 Connection ~ 3700 3300
 $Comp
-L GND #PWR13
+L GND-RESCUE-servo-module-pcb-v1 #PWR13
 U 1 1 55767318
 P 3500 3900
@@
 	3500 3900 3500 3800
 $Comp
-L C C11
+L C-RESCUE-servo-module-pcb-v1 C11
 U 1 1 5576751C
 P 3500 5700
@@
 	3500 5400 3500 5500
 $Comp
-L GND #PWR16
+L GND-RESCUE-servo-module-pcb-v1 #PWR16
 U 1 1 55767524
 P 3500 6000
